Commit message: Update sevenDOF_sword.urdf
prismatic joint nonsense

File: urdf/sevenDOF_sword.urdf (robot description, URDF)
Before this commit: robot SevenDOF, 28 links, 27 joints
Links:
- added link slink
Joints:
- added joint stretch: type prismatic, parent slink, child tip, origin xyz=0 -0.045 0 rpy=0 0 0, axis 0 0 1, limit lower=-0.03 upper=0.15 effort=1000.0 velocity=0.5
- joint attach-cube-left: parent tip -> slink
- joint final: child tip -> slink

Commit message: fixed urdf
realigned joint positions to center the prismatic joint to make the ikin easier

File: urdf/sevenDOF_sword.urdf (robot description, URDF)
Before this commit: robot SevenDOF, 29 links, 28 joints
Joints:
- joint final: origin xyz=0 0.15 0 rpy=1.5708 0 3.1416 -> xyz=0 0.1 0 rpy=1.5708 0 3.1416
- joint stretch: limit lower=-0.03 upper=0.15 effort=1000.0 velocity=0.5 -> lower=-0.09 upper=0.09 effort=1000.0 velocity=0.5; origin xyz=0 -0.045 0 rpy=0 0 0 -> xyz=0 -0.045 0.09 rpy=0 0 0

Commit message: lots of things

File: urdf/sevenDOF_sword.urdf (robot description, URDF)
Before this commit: robot SevenDOF, 29 links, 28 joints
Joints:
- joint stretch: origin xyz=0 -0.045 0.09 rpy=0 0 0 -> xyz=0 -0 0.09 rpy=0 0 0
